File: .experiments/hierarchical_freerouting_demo/parent_preloaded.kicad_pcb (KiCad board)
At the start: 2 copper layers, 120 x 85 mm, 39 parts, among them J1 USB_C, J2 Output, J3 Debug, Q1 FS8205A, U1 USBLC6-2SC6, U2 BQ24072, U3 HY2113-KB5B, U4 MT3608, U5 AP2112K-3.3, U6 LN61CN3302MR-G

Commit message: WIP: subcircuit leaf pipeline - placement, routing, and composition scaffolding
- Expanded solve_subcircuits.py with full leaf solve loop and FreeRouting integration
- Added hierarchy_parser.py for schematic-driven subcircuit tree extraction
- Added subcircuit_solver.py for local placement + Manhattan routing per leaf
- Added subcircuit_board_export.py for mini .kicad_pcb snapshots
- Expanded subcircuit_composer.py with parent composition from rigid children
- Added run_hierarchical_pipeline.py orchestrator
- Added utility scripts: inspect, export, demo
- Improved placement.py outline preservation and force simulation
- Updated AGENTS.md with verification flow
- 6 leaf subcircuits solved (1/6 routed via FreeRouting)
Parts:
- moved BT1 158.6 mm to (221.6, 100.0)
- moved C4 141.1 mm to (207.9, 14.9), turned to 0 degrees
- moved D1 134.2 mm to (205.2, 7.31), turned to -90 degrees
- moved BT2 133.8 mm to (221.6, 75.3)
- moved D2 131.7 mm to (203.3, 11.5), turned to 90 degrees
- moved R8 130.6 mm to (199.8, 15.7), turned to -90 degrees
- moved R7 130.2 mm to (210.5, 10.7), turned to 90 degrees
- moved C3 127.5 mm to (200.2, 5.10)
- moved R6 126.5 mm to (205.8, 3.49), turned to 90 degrees
- moved RT1 121.8 mm to (191.0, 14.7), turned to -90 degrees
- moved U2 120.1 mm to (194.2, 9.18), turned to 90 degrees
- moved R3 118.7 mm to (195.5, 15.6), turned to 90 degrees
- moved C2 116.8 mm to (183.9, 7.84)
- moved R4 112.9 mm to (192.7, 3.70)
- moved R5 105.4 mm to (186.4, 11.5)
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Routing:
- net (no net): track 0.00 -> 699.3 mm
- net /3V3: track 0.00 -> 30.2 mm
- net Net-(D3-A): track 0.00 -> 26.9 mm
- net /VSYS_BOOST: track 0.00 -> 23.2 mm
- net Net-(D2-K): track 0.00 -> 10.7 mm
- net Net-(U2-TMR): track 0.00 -> 8.14 mm
- net Net-(U2-ISET): track 0.00 -> 8.08 mm
- net Net-(D2-A): track 0.00 -> 7.76 mm
- net Net-(D1-A): track 0.00 -> 4.66 mm
- net Net-(U2-ILIM): track 0.00 -> 4.08 mm
Other:
- board size 120 x 85 mm -> 90 x 58 mm
