File: .experiments/subcircuits/subcircuit__8a5edab282/parent_routed.kicad_pcb (KiCad board)
At the start: 2 copper layers, 270.5 x 111.3 mm, 39 parts, among them J1 USB_C, J2 Output, J3 Debug, Q1 FS8205A, U1 USBLC6-2SC6, U2 BQ24072, U3 HY2113-KB5B, U4 MT3608, U5 AP2112K-3.3, U6 LN61CN3302MR-G

Commit message: fix: add board outline rewriting to parent stamp for FreeRouting compatibility
FreeRouting rejects traces outside the board outline. The parent stamp
now rewrites Edge.Cuts to match the composition bounding box so child
copper at composed coordinates is within bounds.

Parent routing now succeeds: FreeRouting routes interconnect nets between
subcircuit blocks on B.Cu (back copper) while preserving all child copper
on F.Cu. Artifacts persisted:
- parent_pre_freerouting.kicad_pcb (stamped with child copper)
- parent_routed.kicad_pcb (with FreeRouting interconnects)
- solved_layout.json (canonical parent artifact)
- metadata.json + debug.json
Routing:
- net (no net): track 1194.9 -> 0.00 mm
- net GND: track 198.6 -> 481.7 mm
- net /VBAT: track 49.8 -> 307.2 mm, vias 0 -> 2
- net /VBUS: track 23.9 -> 239.1 mm, vias 0 -> 2
- net /CELL_NEG: track 19.3 -> 204.4 mm
- net /EN: track 40.7 -> 206.6 mm, vias 0 -> 1
- net Net-(U4-FB): track 11.5 -> 123.1 mm, vias 0 -> 2
- net /5V: track 39.9 -> 133.8 mm
- net /NTC_SENSE: track 19.5 -> 103.0 mm
- net /CHG_N: track 17.4 -> 97.3 mm
- net /VSYS: track 25.6 -> 103.4 mm, vias 0 -> 2

Commit message: feat: unified hierarchical solver (solve_hierarchy.py)
Single-command entry point for the full subcircuit pipeline:
  python3 solve_hierarchy.py LLUPS.kicad_sch --pcb LLUPS.kicad_pcb --route

Phase 1: Solve leaf subcircuits (delegates to solve_subcircuits.py)
  - 6 leaves solved and routed via FreeRouting
  - Canonical copper persisted in solved_layout.json

Phase 2: Compose and route parent (delegates to compose_subcircuits.py)
  - Grid layout of 6 children with 5mm spacing
  - Child copper preserved on stamped parent board
  - FreeRouting routes interconnect nets between subcircuits
  - Parent artifact persisted with full copper

Flags: --skip-leaves, --leaf-only, --rounds, --mode, --spacing-mm, --jar
Full pipeline completes in ~4 minutes (with routing)
Skip-leaves mode completes in ~28 seconds
Parts:
- moved C3 17.5 mm to (206.6, 4.00)
- moved R8 14.9 mm to (193.6, 13.0)
- moved RT1 14.8 mm to (193.5, 17.0), turned to -90 degrees
- moved C2 13.9 mm to (193.3, 9.00), turned to 180 degrees
- moved R7 11.7 mm to (205.4, 12.0)
- moved R3 11.6 mm to (196.6, 4.00), turned to -90 degrees
- moved R4 8.83 mm to (202.6, 8.00), turned to 180 degrees
- moved C4 6.58 mm to (192.6, 5.00)
- moved R6 5.10 mm to (197.8, 8.00), turned to 0 degrees
- moved R9 5.01 mm to (116.5, 8.00), turned to 0 degrees
- moved D2 4.51 mm to (207.6, 8.00), turned to 180 degrees
- moved D1 4.12 mm to (201.6, 4.00)
- moved R5 3.46 mm to (209.9, 12.0)
- moved R11 3.11 mm to (116.6, 12.0), turned to 0 degrees
- moved U2 1.14 mm to (199.4, 14.0), turned to 90 degrees
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Routing:
- net /VSYS: track 103.4 -> 143.5 mm, vias 2 -> 0
- net /EN: track 206.6 -> 184.9 mm, vias 1 -> 0
- net /NTC_SENSE: track 103.0 -> 81.8 mm
- net Net-(D1-A): track 26.1 -> 7.80 mm
- net /VBUS: track 239.1 -> 224.9 mm
- net Net-(U2-ILIM): track 18.5 -> 6.16 mm, vias 2 -> 0
- net /5V: track 133.8 -> 122.2 mm, vias 1 -> 0
- net /CHG_N: track 97.3 -> 88.7 mm, vias 2 -> 1
- net Net-(U4-FB): track 123.1 -> 131.2 mm
- net /VBAT: track 307.2 -> 299.4 mm
- net Net-(U2-ISET): track 9.04 -> 14.9 mm, vias 2 -> 0
- net Net-(U2-TMR): track 11.0 -> 14.8 mm, vias 0 -> 2
- net /3V3: track 33.0 -> 36.0 mm, vias 0 -> 2
- net Net-(D2-K): track 9.01 -> 11.3 mm, vias 2 -> 0
- net Net-(D2-A): track 8.83 -> 6.52 mm
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